File: minimal_lt8304/minimal_lt8304.kicad_pcb (KiCad board)
At the start: 4 copper layers, 63.9 x 22.9 mm, 39 parts, among them J1 FW-02-03-G-D-085-155, J2 FW-02-03-G-D-085-155, J3 FW-02-03-G-D-085-155, J4 FW-02-03-G-D-085-155, T1 750315836, U1 LT8304IS8E-PBF

Commit message: Small project update
Parts:
- added D4: 100.0 V, diode_footprints:SOD123W, F.Cu at (181.5, 103.1)
- added JP2: SolderJumper_3_Open, solder_jumper_footprints:SolderJumper-3_P1.3mm_Bridged_1_2_RoundedPad1.0x1.5mm_NumberLabels, F.Cu at (186.4, 102.9)
- moved C6 1.78 mm to (182.9, 109.2)
- moved C7 1.78 mm to (182.9, 118.5)
Connections:
- J1 pad 1: /VOUT -> /VOUT_SELECTED
- J1 pad 3: /VOUT -> /VOUT_SELECTED
- TP3 pad 1: /VOUT -> /VOUT_SELECTED
Routing:
- net GNDA: vias 70 -> 64
- net /VOUT_SELECTED: vias 0 -> 6
- net /VOUT: vias 35 -> 21
- added copper zone on F.Cu, net /VOUT_SELECTED
- added copper zone on In1.Cu, net /VOUT_SELECTED
- added copper zone on F.Cu, net Net-(JP2-A)

Commit message: update project
Parts:
- removed J3, J4: FW-02-03-G-D-085-155, connector_footprints:FW-02-03-G-D-085-155
- removed MB3, MB4: mouse-bite-midle-50mil-200mil, mouse_bite_footprints:mouse-bite-midle-50mil-200mil
- removed TP5, TP6, TP7, TP8: TestPoint, test_point_footprints:TestPoint_THTPad_Castelated
- moved J1 6.98 mm to (195.5, 112.1)
- moved MB2 6.98 mm to (192.4, 112.1)
- moved TP3 6.98 mm to (191.7, 111.4)
- moved TP4 6.98 mm to (191.7, 112.7)
- moved FID2 3.81 mm to (150.4, 101.9)
- moved MB1 3.81 mm to (146.6, 103.8)
- moved TP1 3.81 mm to (147.3, 104.4)
- moved TP2 3.81 mm to (147.3, 103.2)
- moved J2 3.80 mm to (142.2, 103.8)
Routing:
- net GNDA: vias 64 -> 52
- net GND: vias 64 -> 51
- net /VIN: vias 32 -> 28
Other:
- board size 63.9 x 22.9 mm -> 60.1 x 22.9 mm

Commit message: update project
Parts:
- moved FID2 1.91 mm to (152.3, 101.9)
- moved J2 1.91 mm to (144.1, 103.8)
- moved MB1 1.91 mm to (148.5, 103.8)
- moved TP1 1.91 mm to (149.2, 104.4)
- moved TP2 1.91 mm to (149.2, 103.2)
- moved C4 1.42 mm to (143.5, 113.5), turned to -90 degrees
- moved R6 1.40 mm to (146.9, 119.4)
- moved R3 1.07 mm to (147.8, 117.5), turned to -90 degrees
- moved C1 0.37 mm to (148.8, 121.5)
Routing:
- net GND: vias 51 -> 47
- net /VIN: vias 28 -> 27
Other:
- board size 60.1 x 22.9 mm -> 58.2 x 22.9 mm

Commit message: development backup
Parts:
- moved FID3 49.8 mm to (140.7, 122.5)
- moved J1 8.91 mm to (196.2, 121.0), turned to -90 degrees
- moved MB2 8.89 mm to (192.4, 121.0)
- moved TP3 8.89 mm to (191.7, 120.3)
- moved TP4 8.89 mm to (191.7, 121.6)
- moved FID2 2.17 mm to (150.2, 101.7)
Connections:
- J1 pad 2: GNDA -> /VOUT_SELECTED
- J1 pad 3: /VOUT_SELECTED -> GNDA
Routing:
- net /VIN: vias 27 -> 26
Other:
- board size 58.2 x 22.9 mm -> 61 x 22.9 mm
