File: minimal_lt8304/minimal_lt8304.kicad_pcb (KiCad board)
At the start: 4 copper layers, 61 x 22.9 mm, 33 parts, among them J1 FW-02-03-G-D-085-155, J2 FW-02-03-G-D-085-155, T1 750315836, U1 LT8304IS8E-PBF

Commit message: development backup
Parts:
- added REF**: OSHW-Logo_5.7x6mm_SilkScreen, Symbol:OSHW-Logo_5.7x6mm_SilkScreen, F.Cu at (158.7, 103.3)
- added REF**: KiCad-Logo2_5mm_SilkScreen, Symbol:KiCad-Logo2_5mm_SilkScreen, F.Cu at (166.5, 103.3)
